File: hardware/strain_guage_PCB/_autosave-strain_guage.kicad_pcb (KiCad board)
At the start: 4 copper layers, 140.3 x 89.5 mm, 93 parts, among them IC1 STM32C091CBT6, J2 Conn_02x05_Odd_Even, J3 Screw_Terminal_01x03, SW1 SW_Push, U1 MCP3561-E/ST, U10 MCP2221A-I/SL, U11 LM2664M6X/NOPB, U2 OP177GPZ, U3 OP177GPZ, U4 OP177GPZ, U5 AD630ARZ, U6 OPA2187IDR, U7 OP177GPZ, U8 AD9833BRMZ, U9 MIC5365-3.3YC5-TR

Commit message: Small changes to improve manufacturability
Parts:
- U2, U3, U4, U7: footprint Package_DIP:DIP-8_W7.62mm -> OP177GPZ:DIP794W56P254L959H533Q8N
- moved U3 5.38 mm to (120.5, 93.6)
- moved U7 5.35 mm to (108.3, 69.8)
- moved U2 5.23 mm to (104.5, 93.4)
- moved U4 5.21 mm to (137.3, 93.6)
Routing:
- net Net-(R11-Pad2): track 19.9 -> 19.2 mm
