File: hardware/strain_guage_PCB/strain_guage.kicad_sch (KiCad schematic)
At the start: 97 parts, among them IC1 STM32C091CBT6, J2 Conn_02x05_Odd_Even, J3 Screw_Terminal_01x03, SW1 SW_Push, U1 MCP3561-E/ST, U10 MCP2221A-I/SL, U11 LM2664M6X/NOPB, U2 OP177GPZ, U3 OP177GPZ, U4 OP177GPZ, U5 AD630ARZ, U6 OPA2187IDR, U7 OP177GPZ, U8 AD9833BRMZ, U9 MIC5365-3.3YC5-TR

Commit message: PCB Revision + BOM Update
Footprints for Op-Amps were corrected, package size for R22 was updated. PCB Layout and Tracing marginally modified
Parts:
- R22: footprint Resistor_SMD:R_0201_0603Metric -> Resistor_SMD:R_0402_1005Metric
Changed lines of the file:
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@@
 			)
 		)
-		(property "Footprint" "Resistor_SMD:R_0201_0603Metric"
+		(property "Footprint" "Resistor_SMD:R_0402_1005Metric"
 			(at 325.882 190.5 90)
 			(effects

Commit message: Op-Amp footprints updated
Parts:
- U2, U3, U4, U7: footprint Package_DIP:DIP-8-16_W7.62mm -> Package_DIP:DIP-8_W7.62mm
Changed lines of the file:
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@@
 			)
 		)
-		(property "Footprint" "Package_DIP:DIP-8-16_W7.62mm"
+		(property "Footprint" "Package_DIP:DIP-8_W7.62mm"
 			(at 251.46 68.58 0)
 			(effects
@@
 			)
 		)
-		(property "Footprint" "Package_DIP:DIP-8-16_W7.62mm"
+		(property "Footprint" "Package_DIP:DIP-8_W7.62mm"
 			(at 212.09 148.59 0)
 			(effects
@@
 			)
 		)
-		(property "Footprint" "Package_DIP:DIP-8-16_W7.62mm"
+		(property "Footprint" "Package_DIP:DIP-8_W7.62mm"
 			(at 196.85 50.8 0)
 			(effects
@@
 			)
 		)
-		(property "Footprint" "Package_DIP:DIP-8-16_W7.62mm"
+		(property "Footprint" "Package_DIP:DIP-8_W7.62mm"
 			(at 196.85 88.9 0)
 			(effects

Commit message: Small changes to improve manufacturability
Parts:
- U2, U3, U4, U7: footprint Package_DIP:DIP-8_W7.62mm -> OP177GPZ:DIP794W56P254L959H533Q8N
Changed lines of the file:
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@@
 			)
 		)
-		(property "Footprint" "Package_DIP:DIP-8_W7.62mm"
+		(property "Footprint" "OP177GPZ:DIP794W56P254L959H533Q8N"
 			(at 251.46 68.58 0)
 			(effects
@@
 			)
 		)
-		(property "Footprint" "Package_DIP:DIP-8_W7.62mm"
+		(property "Footprint" "OP177GPZ:DIP794W56P254L959H533Q8N"
 			(at 212.09 148.59 0)
 			(effects
@@
 			)
 		)
-		(property "Footprint" "Package_DIP:DIP-8_W7.62mm"
+		(property "Footprint" "OP177GPZ:DIP794W56P254L959H533Q8N"
 			(at 196.85 50.8 0)
 			(effects
@@
 			)
 		)
-		(property "Footprint" "Package_DIP:DIP-8_W7.62mm"
+		(property "Footprint" "OP177GPZ:DIP794W56P254L959H533Q8N"
 			(at 196.85 88.9 0)
 			(effects
